Commit message: Added robot_v1 to rviz, gazebo and changed visual

File: catkin_ws/src/fyp_sim/urdf/robot_platform.urdf (robot description, URDF)
Before this commit: robot robot_platform, 5 links, 4 joints
Links:
- removed link link_2
- removed link link_3
- removed link link_4
- added link dummy
Joints:
- removed joint joint_2
- removed joint joint_3
- removed joint joint_4
- added joint dummy_joint: type fixed, parent dummy, child link_0
