Commit message: Added controllers, fixed URDF, added GPS and tested

File: catkin_ws/src/fyp_sim/urdf/materials.xacro (robot description, xacro)
@@ -1,4 +1,4 @@
 <?xml version="1.0" encoding="utf-8"?>
-<robot name="robot_platform" xmlns:xacro="http://www.ros.org/wiki/xacro">
+<robot name="robot_platform_material" xmlns:xacro="http://www.ros.org/wiki/xacro">
   <material name="black">
     <color rgba="0.0 0.0 0.0 1.0" />

File: catkin_ws/src/fyp_sim/urdf/robot.gazebo.xacro (robot description, xacro)
@@ -1,4 +1,4 @@
 <?xml version="1.0"?>
-<robot name="robot_platform" xmlns:xacro="http://www.ros.org/wiki/xacro">
+<robot name="robot_platform_gazebo" xmlns:xacro="http://www.ros.org/wiki/xacro">
   <gazebo reference="chassis">
     <material>Gazebo/Grey</material>
@@ -22,4 +22,22 @@
     <material>Gazebo/Black</material>
   </gazebo>
+  <gazebo>
+    <plugin name="gazebo_ros_control" filename="libgazebo_ros_control.so">
+      <robotNamespace>/robot_platform_control</robotNamespace>
+      <!-- <robotSimType>gazebo_ros_control/DefaultRobotHWSim</robotSimType> -->
+    </plugin>
+  </gazebo>
+  <!-- GPS plugin -->
+  <gazebo>
+    <plugin name="gps_controller" filename="libhector_gazebo_ros_gps.so">
+      <alwaysOn>true</alwaysOn>
+      <updateRate>10.0</updateRate>
+      <bodyName>chassis</bodyName>
+      <topicName>gpsfix</topicName>
+      <velocityGaussianNoise>0.1 0.1 0.1</velocityGaussianNoise>
+      <status>1</status>
+      <service>2</service>
+    </plugin>
+  </gazebo>
   <!-- <gazebo>
     <plugin filename="libgazebo_ros_diff_drive.so" name="differential_drive_controller">

File: catkin_ws/src/fyp_sim/urdf/robot.xacro (robot description, xacro)
@@ -1,9 +1,8 @@
 <?xml version="1.0" encoding="utf-8"?>
-<robot name="robot_platform" xmlns:xacro="http://www.ros.org/wiki/xacro">
+<robot name="robot_platform_urdf" xmlns:xacro="http://www.ros.org/wiki/xacro">
   <!-- <xacro:include filename="$(find fyp_sim)/urdf/materials.xacro"/> -->
-  <xacro:include filename="$(find fyp_sim)/urdf/robot.gazebo"/>
+  <xacro:include filename="$(find fyp_sim)/urdf/robot.gazebo.xacro"/>
   <!-- dummy link -->
-  <link name="dummy">
-  </link>
+  <link name="base_footprint"/>
   <!-- chassis -->
   <link name="chassis">
@@ -84,4 +83,14 @@
           filename="package://fyp_sim/meshes/back_wheel.stl" scale="0.01 0.01 0.01"/>
       </geometry>
+      <surface>
+        <friction>
+          <ode>
+            <mu>0.8</mu>
+            <mu2>0.8</mu2>
+            <slip1>1.0</slip1>
+            <slip2>1.0</slip2>
+          </ode>
+        </friction>
+      </surface>
     </collision>
   </link>
@@ -124,4 +133,14 @@
           filename="package://fyp_sim/meshes/back_wheel.stl" scale="0.01 0.01 0.01"/>
       </geometry>
+      <surface>
+        <friction>
+          <ode>
+            <mu>0.8</mu>
+            <mu2>0.8</mu2>
+            <slip1>1.0</slip1>
+            <slip2>1.0</slip2>
+          </ode>
+        </friction>
+      </surface>
     </collision>
   </link>
@@ -244,4 +263,14 @@
           filename="package://fyp_sim/meshes/front_wheel.stl" scale="0.01 0.01 0.01"/>
       </geometry>
+      <surface>
+        <friction>
+          <ode>
+            <mu>0.8</mu>
+            <mu2>0.8</mu2>
+            <slip1>1.0</slip1>
+            <slip2>1.0</slip2>
+          </ode>
+        </friction>
+      </surface>
     </collision>
   </link>
@@ -284,12 +313,22 @@
           filename="package://fyp_sim/meshes/front_wheel.stl" scale="0.01 0.01 0.01"/>
       </geometry>
-    </collision>
-  </link>
-  <joint name="dummy_joint" type="fixed">
-    <origin
-      xyz="0 0 0.23487"
+      <surface>
+        <friction>
+          <ode>
+            <mu>0.8</mu>
+            <mu2>0.8</mu2>
+            <slip1>1.0</slip1>
+            <slip2>1.0</slip2>
+          </ode>
+        </friction>
+      </surface>
+    </collision>
+  </link>
+  <joint name="base_joint" type="fixed">
+    <origin
+      xyz="0 0 0.22987"
       rpy="0 0 0" />
     <parent
-      link="dummy" />
+      link="base_footprint" />
     <child
       link="chassis" />
@@ -298,5 +337,5 @@
     type="continuous">
     <origin
-      xyz="0.23591 -0.24479 -0.07497"
+      xyz="0.23591 -0.245 -0.06987"
       rpy="${pi/2} 0 0" />
     <parent
@@ -310,5 +349,5 @@
     type="continuous">
     <origin
-      xyz="0.23591 0.24521 -0.07487"
+      xyz="0.23591 0.245 -0.06987"
       rpy="${-pi/2} 0 0" />
     <parent
@@ -320,7 +359,8 @@
   </joint>
   <joint name="front_LW_con_joint"
-    type="continuous">
-    <origin
-      xyz="-0.35409 -0.21979 0.01513"
+    type="revolute">
+    <limit effort="30" velocity="4.0" lower="-3.14159" upper="3.14159"/>
+    <origin
+      xyz="-0.35409 -0.22 0.02013"
       rpy="0 0 ${pi/2}" />
     <parent
@@ -332,7 +372,8 @@
   </joint>
   <joint name="front_RW_con_joint"
-    type="continuous">
-    <origin
-      xyz="-0.35409 0.22021 0.01513"
+    type="revolute">
+    <limit effort="30" velocity="4.0" lower="-3.14159" upper="3.14159"/>
+    <origin
+      xyz="-0.35409 0.22 0.02013"
       rpy="0 0 ${pi/2}" />
     <parent
@@ -346,8 +387,8 @@
     type="continuous">
     <origin
-      xyz="-0.35409 0.22521 -0.13487"
-      rpy="${-pi/2} 0 0" />
-    <parent
-      link="chassis" />
+      xyz="0 0 -0.15"
+      rpy="0 ${pi/2} 0" />
+    <parent
+      link="front_wheel_right_connector" />
     <child
       link="front_wheel_right" />
@@ -355,11 +396,12 @@
       xyz="0 0 1" />
   </joint>
+<!-- "-0.35409 -0.22 -0.13487" -->
   <joint name="front_LW_joint"
     type="continuous">
     <origin
-      xyz="-0.35409 -0.21479 -0.13487"
-      rpy="${-pi/2} 0 0" />
-    <parent
-      link="chassis"/>
+      xyz="0 0 -0.15"
+      rpy="0 ${-pi/2} 0" />
+    <parent
+      link="front_wheel_left_connector"/>
     <child
       link="front_wheel_left" />
@@ -367,3 +409,43 @@
       xyz="0 0 1" />
   </joint>
+  <transmission name="back_LW_transmission">
+    <type>transmission_interface/SimpleTransmission</type>
+    <joint name="back_LW_joint">
+      <hardwareInterface>hardware_interface/EffortJointInterface</hardwareInterface>
+    </joint>
+    <actuator name="back_LW_motor">
+      <mechanicalReduction>1</mechanicalReduction>
+      <hardwareInterface>EffortJointInterface</hardwareInterface>
+    </actuator>
+  </transmission>
+  <transmission name="back_RW_transmission">
+    <type>transmission_interface/SimpleTransmission</type>
+    <joint name="back_RW_joint">
+      <hardwareInterface>hardware_interface/EffortJointInterface</hardwareInterface>
+    </joint>
+    <actuator name="back_RW_motor">
+      <mechanicalReduction>1</mechanicalReduction>
+      <hardwareInterface>EffortJointInterface</hardwareInterface>
+    </actuator>
+  </transmission>
+  <transmission name="front_RW_con_transmission">
+    <type>transmission_interface/SimpleTransmission</type>
+    <joint name="front_RW_con_joint">
+      <hardwareInterface>hardware_interface/EffortJointInterface</hardwareInterface>
+    </joint>
+    <actuator name="front_RW_con_motor">
+      <mechanicalReduction>1</mechanicalReduction>
+      <hardwareInterface>EffortJointInterface</hardwareInterface>
+    </actuator>
+  </transmission>
+  <transmission name="front_LW_con_transmission">
+    <type>transmission_interface/SimpleTransmission</type>
+    <joint name="front_LW_con_joint">
+      <hardwareInterface>hardware_interface/EffortJointInterface</hardwareInterface>
+    </joint>
+    <actuator name="front_LW_con_motor">
+      <mechanicalReduction>1</mechanicalReduction>
+      <hardwareInterface>EffortJointInterface</hardwareInterface>
+    </actuator>
+  </transmission>
 </robot>
