Commit message: added navigation, movebase, removed steering

File: catkin_ws/src/fyp_sim/urdf/robot.gazebo.xacro (robot description, xacro)
@@ -41,14 +41,75 @@
   </gazebo>
   <!-- IMU plugin -->
+  <!-- <gazebo>
+    <plugin filename="libgazebo_ros_imu.so" name="imu_plugin">
+      <alwaysOn>true</alwaysOn>
+      <topicName>/imu</topicName>
+      <bodyName>base_footprint</bodyName>
+      <updateRate>10.0</updateRate>
+      <gaussianNoise>0.0</gaussianNoise>
+      <xyzOffset>0 0 0</xyzOffset>
+      <rpyOffset>0 0 0</rpyOffset>
+    </plugin>
+  </gazebo> -->
   <gazebo>
-    <plugin name="imu_plugin" filename="libgazebo_ros_imu.so">
-      <alwaysOn>true</alwaysOn>
+    <plugin filename="libhector_gazebo_ros_imu.so" name="imu_plugin">
+      <topicName>/imu</topicName>
       <bodyName>base_footprint</bodyName>
-      <topicName>imu</topicName>
-      <serviceName>imu_service</serviceName>
+      <updateRate>10.0</updateRate>
       <gaussianNoise>0.0</gaussianNoise>
-      <updateRate>20.0</updateRate>
+      <rpyOffset>0 0 0</rpyOffset>
     </plugin>
   </gazebo>
+  <!-- <gazebo reference="imu_link">
+  <gravity>true</gravity>
+    <sensor name="imu_sensor" type="imu">
+      <always_on>true</always_on>
+      <update_rate>10</update_rate>
+      <visualize>true</visualize>
+      <plugin filename="libgazebo_ros_imu_sensor.so" name="imu_plugin">
+        <topicName>/imuu</topicName>
+        <bodyName>lidar</bodyName>
+        <updateRateHZ>10</updateRateHZ>
+        <gaussianNoise>0.0</gaussianNoise>
+        <xyzOffset>0 0 0</xyzOffset>
+        <rpyOffset>0 0 0</rpyOffset>
+        <frameName>lidar</frameName>
+        <initialOrientationAsReference>false</initialOrientationAsReference>
+      </plugin>
+      <pose>0 0 0 0 0 0</pose>
+    </sensor>
+  </gazebo> -->
+  <!-- Laser plugin -->
+  <!-- <gazebo reference="lidar">
+      <sensor type="gpu_ray" name="lidar_sensor">
+        <pose>0 0 0 0 0 0</pose>
+        <visualize>false</visualize>
+        <update_rate>40</update_rate>
+        <ray>
+          <scan>
+            <horizontal>
+              <samples>720</samples>
+              <resolution>1</resolution>
+              <min_angle>-3.141592</min_angle>
+              <max_angle>3.141592</max_angle>
+            </horizontal>
+          </scan>
+          <range>
+            <min>0.10</min>
+            <max>9</max>
+            <resolution>0.01</resolution>
+          </range>
+          <noise>
+            <type>gaussian</type>
+            <mean>0.0</mean>
+            <stddev>0.01</stddev>
+          </noise>
+        </ray>
+        <plugin name="gazebo_ros_head_hokuyo_controller" filename="libgazebo_ros_gpu_laser.so">
+          <topicName>/laser/scan</topicName>
+          <frameName>lidar</frameName>
+        </plugin>
+      </sensor>
+    </gazebo> -->
   <!-- <gazebo>
     <plugin filename="libgazebo_ros_diff_drive.so" name="differential_drive_controller">

File: catkin_ws/src/fyp_sim/urdf/robot.xacro (robot description, xacro)
@@ -12,5 +12,5 @@
         rpy="0 0 0" />
       <mass
-        value="6.52316744505344" />
+        value="28" />
       <inertia
         ixx="0.0385919077427861"
@@ -232,12 +232,12 @@
         rpy="0 0 0" />
       <mass
-        value="0.853825179360506" />
-      <inertia
-        ixx="0.00259189846991135"
-        ixy="2.99550060933435E-17"
-        ixz="2.12803718614051E-20"
-        iyy="0.00473869680320454"
-        iyz="-7.59085432106584E-18"
-        izz="0.00237094198835257" />
+        value="1" />
+        <inertia
+          ixx="1E-3"
+          ixy="0"
+          ixz="0"
+          iyy="1E-3"
+          iyz="0"
+          izz="1E-3" />
     </inertial>
     <visual>
@@ -268,6 +268,6 @@
             <mu>0.8</mu>
             <mu2>0.8</mu2>
-            <slip1>1.0</slip1>
-            <slip2>1.0</slip2>
+            <!-- <slip1>1.0</slip1>
+            <slip2>1.0</slip2> -->
           </ode>
         </friction>
@@ -282,12 +282,12 @@
         rpy="0 0 0" />
       <mass
-        value="0.853825179360506" />
-      <inertia
-        ixx="0.00259189846991135"
-        ixy="2.99550060933435E-17"
-        ixz="2.12803718614051E-20"
-        iyy="0.00473869680320454"
-        iyz="-7.59085432106584E-18"
-        izz="0.00237094198835257" />
+        value="1" />
+      <inertia
+        ixx="1E-3"
+        ixy="0"
+        ixz="0"
+        iyy="1E-3"
+        iyz="0"
+        izz="1E-3" />
     </inertial>
     <visual>
@@ -318,6 +318,6 @@
             <mu>0.8</mu>
             <mu2>0.8</mu2>
-            <slip1>1.0</slip1>
-            <slip2>1.0</slip2>
+            <!-- <slip1>1.0</slip1>
+            <slip2>1.0</slip2> -->
           </ode>
         </friction>
@@ -325,4 +325,41 @@
     </collision>
   </link>
+  <link name="lidar">
+    <inertial>
+      <origin
+        xyz="0 0 0"
+        rpy="0 0 0" />
+      <mass
+        value="0.3" />
+      <inertia
+        ixx="0"
+        ixy="0"
+        ixz="0"
+        iyy="0"
+        iyz="0"
+        izz="0.01" />
+    </inertial>
+    <visual>
+      <origin
+        xyz="0 0 0"
+        rpy="0 0 0" />
+      <geometry>
+        <cylinder radius="0.04" length="0.04"/>
+      </geometry>
+      <material
+        name="cylinder_material">
+        <color
+          rgba="0.0 0.0 0.0 1.0" />
+      </material>
+    </visual>
+    <collision>
+      <origin
+        xyz="0 0 0"
+        rpy="0 0 0" />
+        <geometry>
+          <cylinder radius="0.04" length="0.04"/>
+        </geometry>
+    </collision>
+  </link>
   <joint name="base_joint" type="fixed">
     <origin
@@ -333,4 +370,13 @@
     <child
       link="chassis" />
+  </joint>
+  <joint name="lidar_joint" type="fixed">
+    <origin
+      xyz="-0.29 0 0.29"
+      rpy="0 0 0" />
+    <parent
+      link="chassis" />
+    <child
+      link="lidar" />
   </joint>
   <joint name="back_LW_joint"
@@ -345,4 +391,5 @@
     <axis
       xyz="0 0 1" />
+      <dynamics damping="0.4" friction="0.4"/>
   </joint>
   <joint name="back_RW_joint"
@@ -357,8 +404,9 @@
     <axis
       xyz="0 0 -1" />
+      <dynamics damping="0.4" friction="0.4"/>
   </joint>
   <joint name="front_LW_con_joint"
-    type="revolute">
-    <limit effort="30" velocity="${pi/3}" lower="${-pi/2}" upper="${pi/2}"/>
+    type="continuous">
+    <!-- <limit effort="30" velocity="${pi/3}" lower="${-pi/2}" upper="${pi/2}"/> -->
     <origin
       xyz="-0.35409 -0.22 0.02013"
@@ -370,8 +418,9 @@
     <axis
       xyz="0 0 1" />
+      <dynamics friction="0.1"/>
   </joint>
   <joint name="front_RW_con_joint"
-    type="revolute">
-    <limit effort="30" velocity="${pi/3}" lower="${-pi/2}" upper="${pi/2}"/>
+    type="continuous">
+    <!-- <limit effort="30" velocity="${pi/3}" lower="${-pi/2}" upper="${pi/2}"/> -->
     <origin
       xyz="-0.35409 0.22 0.02013"
@@ -383,4 +432,5 @@
     <axis
       xyz="0 0 1" />
+      <dynamics friction="0.1"/>
   </joint>
   <joint name="front_RW_joint"

Commit message: last update before reversing

File: catkin_ws/src/fyp_sim/urdf/robot.gazebo.xacro (robot description, xacro)
@@ -60,4 +60,40 @@
       <rpyOffset>0 0 0</rpyOffset>
     </plugin>
+  </gazebo>
+  <gazebo reference="back_wheel_right">
+    <kp>1000000.0</kp>
+    <kd>100.0</kd>
+    <mu1>1.5</mu1>
+    <mu2>1.5</mu2>
+    <fdir1>1 0 0</fdir1>
+    <maxVel>1.0</maxVel>
+    <minDepth>0.00</minDepth>
+  </gazebo>
+  <gazebo reference="back_wheel_left">
+    <kp>1000000.0</kp>
+    <kd>100.0</kd>
+    <mu1>1.5</mu1>
+    <mu2>1.5</mu2>
+    <fdir1>1 0 0</fdir1>
+    <maxVel>1.0</maxVel>
+    <minDepth>0.00</minDepth>
+  </gazebo>
+  <gazebo reference="front_wheel_right">
+    <kp>1000000.0</kp>
+    <kd>100.0</kd>
+    <mu1>1.5</mu1>
+    <mu2>1.5</mu2>
+    <fdir1>1 0 0</fdir1>
+    <maxVel>1.0</maxVel>
+    <minDepth>0.00</minDepth>
+  </gazebo>
+  <gazebo reference="front_wheel_left">
+    <kp>1000000.0</kp>
+    <kd>100.0</kd>
+    <mu1>1.5</mu1>
+    <mu2>1.5</mu2>
+    <fdir1>1 0 0</fdir1>
+    <maxVel>1.0</maxVel>
+    <minDepth>0.00</minDepth>
   </gazebo>
   <!-- <gazebo reference="imu_link">

File: catkin_ws/src/fyp_sim/urdf/robot.xacro (robot description, xacro)
@@ -52,184 +52,4 @@
         rpy="0 0 0" />
       <mass
-        value="0.853825179360506" />
-      <inertia
-        ixx="0.00259189846991135"
-        ixy="2.99550060933435E-17"
-        ixz="2.12803718614051E-20"
-        iyy="0.00473869680320454"
-        iyz="-7.59085432106584E-18"
-        izz="0.00237094198835257" />
-    </inertial>
-    <visual>
-      <origin
-        xyz="0 0 0"
-        rpy="0 0 0" />
-      <geometry>
-        <mesh
-          filename="package://fyp_sim/meshes/back_wheel.stl" scale="0.01 0.01 0.01"/>
-      </geometry>
-      <material
-        name="back_wheel_left_material">
-        <color
-          rgba="0.0 0.0 0.0 1.0" />
-      </material>
-    </visual>
-    <collision name="back_wheel_left_collision">
-      <origin
-        xyz="0 0 0"
-        rpy="0 0 0" />
-      <geometry>
-        <mesh
-          filename="package://fyp_sim/meshes/back_wheel.stl" scale="0.01 0.01 0.01"/>
-      </geometry>
-      <surface>
-        <friction>
-          <ode>
-            <mu>0.8</mu>
-            <mu2>0.8</mu2>
-            <slip1>1.0</slip1>
-            <slip2>1.0</slip2>
-          </ode>
-        </friction>
-      </surface>
-    </collision>
-  </link>
-  <!-- back wheel right -->
-  <link name="back_wheel_right">
-    <inertial>
-      <origin
-        xyz="0 0 0"
-        rpy="0 0 0" />
-      <mass
-        value="0.853825179360506" />
-      <inertia
-        ixx="0.00259189846991135"
-        ixy="2.99550060933435E-17"
-        ixz="2.12803718614051E-20"
-        iyy="0.00473869680320454"
-        iyz="-7.59085432106584E-18"
-        izz="0.00237094198835257" />
-    </inertial>
-    <visual>
-      <origin
-        xyz="0 0 0"
-        rpy="0 0 0" />
-      <geometry>
-        <mesh
-          filename="package://fyp_sim/meshes/back_wheel.stl" scale="0.01 0.01 0.01"/>
-      </geometry>
-      <material
-        name="back_wheel_right_material">
-        <color
-          rgba="0.0 0.0 0.0 1.0" />
-      </material>
-    </visual>
-    <collision name="back_wheel_right_collision">
-      <origin
-        xyz="0 0 0"
-        rpy="0 0 0" />
-      <geometry>
-        <mesh
-          filename="package://fyp_sim/meshes/back_wheel.stl" scale="0.01 0.01 0.01"/>
-      </geometry>
-      <surface>
-        <friction>
-          <ode>
-            <mu>0.8</mu>
-            <mu2>0.8</mu2>
-            <slip1>1.0</slip1>
-            <slip2>1.0</slip2>
-          </ode>
-        </friction>
-      </surface>
-    </collision>
-  </link>
-  <!-- front wheel left connector -->
-  <link name="front_wheel_left_connector">
-    <inertial>
-      <origin
-        xyz="0 0 0"
-        rpy="0 0 0" />
-      <mass
-        value="0.853825179360506" />
-      <inertia
-        ixx="0.00259189846991135"
-        ixy="2.99550060933435E-17"
-        ixz="2.12803718614051E-20"
-        iyy="0.00473869680320454"
-        iyz="-7.59085432106584E-18"
-        izz="0.00237094198835257" />
-    </inertial>
-    <visual>
-      <origin
-        xyz="0 0 0"
-        rpy="0 0 0" />
-      <geometry>
-        <mesh
-          filename="package://fyp_sim/meshes/front_wheel_connector.stl" scale="0.01 0.01 0.01"/>
-      </geometry>
-      <material
-        name="front_wheel_left_connector_material">
-        <color
-          rgba="0.203125 0.238281 0.285156 1.0" />
-      </material>
-    </visual>
-    <collision name="front_wheel_left_connector_collision">
-      <origin
-        xyz="0 0 0"
-        rpy="0 0 0" />
-      <geometry>
-        <mesh
-          filename="package://fyp_sim/meshes/front_wheel_connector.stl" scale="0.01 0.01 0.01"/>
-      </geometry>
-    </collision>
-  </link>
-  <!-- front wheel right connector -->
-  <link name="front_wheel_right_connector">
-    <inertial>
-      <origin
-        xyz="0 0 0"
-        rpy="0 0 0" />
-      <mass
-        value="0.853825179360506" />
-      <inertia
-        ixx="0.00259189846991135"
-        ixy="2.99550060933435E-17"
-        ixz="2.12803718614051E-20"
-        iyy="0.00473869680320454"
-        iyz="-7.59085432106584E-18"
-        izz="0.00237094198835257" />
-    </inertial>
-    <visual>
-      <origin
-        xyz="0 0 0"
-        rpy="0 0 0" />
-      <geometry>
-        <mesh
-          filename="package://fyp_sim/meshes/front_wheel_connector.stl" scale="0.01 0.01 0.01"/>
-      </geometry>
-      <material
-        name="front_wheel_right_connector_material">
-        <color
-          rgba="0.203125 0.238281 0.285156 1.0" />
-      </material>
-    </visual>
-    <collision name="front_wheel_right_connector_collision">
-      <origin
-        xyz="0 0 0"
-        rpy="0 0 0" />
-      <geometry>
-        <mesh
-          filename="package://fyp_sim/meshes/front_wheel_connector.stl" scale="0.01 0.01 0.01"/>
-      </geometry>
-    </collision>
-  </link>
-  <!-- front wheel right -->
-  <link name="front_wheel_right">
-    <inertial>
-      <origin
-        xyz="0 0 0"
-        rpy="0 0 0" />
-      <mass
         value="1" />
         <inertia
@@ -247,25 +67,25 @@
       <geometry>
         <mesh
-          filename="package://fyp_sim/meshes/front_wheel.stl" scale="0.01 0.01 0.01"/>
-      </geometry>
-      <material
-        name="front_wheel_right_material">
+          filename="package://fyp_sim/meshes/back_wheel.stl" scale="0.01 0.01 0.01"/>
+      </geometry>
+      <material
+        name="back_wheel_left_material">
         <color
           rgba="0.0 0.0 0.0 1.0" />
       </material>
     </visual>
-    <collision name="front_wheel_right_collision">
-      <origin
-        xyz="0 0 0"
-        rpy="0 0 0" />
-      <geometry>
-        <mesh
-          filename="package://fyp_sim/meshes/front_wheel.stl" scale="0.01 0.01 0.01"/>
+    <collision name="back_wheel_left_collision">
+      <origin
+        xyz="0 0 0"
+        rpy="0 0 0" />
+      <geometry>
+        <mesh
+          filename="package://fyp_sim/meshes/back_wheel.stl" scale="0.01 0.01 0.01"/>
       </geometry>
       <surface>
         <friction>
           <ode>
-            <mu>0.8</mu>
-            <mu2>0.8</mu2>
+            <mu>1</mu>
+            <mu2>1</mu2>
             <!-- <slip1>1.0</slip1>
             <slip2>1.0</slip2> -->
@@ -275,4 +95,260 @@
     </collision>
   </link>
+  <!-- back wheel right -->
+  <link name="back_wheel_right">
+    <inertial>
+      <origin
+        xyz="0 0 0"
+        rpy="0 0 0" />
+      <mass
+        value="1" />
+        <inertia
+          ixx="1E-3"
+          ixy="0"
+          ixz="0"
+          iyy="1E-3"
+          iyz="0"
+          izz="1E-3" />
+    </inertial>
+    <visual>
+      <origin
+        xyz="0 0 0"
+        rpy="0 0 0" />
+      <geometry>
+        <mesh
+          filename="package://fyp_sim/meshes/back_wheel.stl" scale="0.01 0.01 0.01"/>
+      </geometry>
+      <material
+        name="back_wheel_right_material">
+        <color
+          rgba="0.0 0.0 0.0 1.0" />
+      </material>
+    </visual>
+    <collision name="back_wheel_right_collision">
+      <origin
+        xyz="0 0 0"
+        rpy="0 0 0" />
+      <geometry>
+        <mesh
+          filename="package://fyp_sim/meshes/back_wheel.stl" scale="0.01 0.01 0.01"/>
+      </geometry>
+      <surface>
+        <friction>
+          <ode>
+            <mu>1</mu>
+            <mu2>1</mu2>
+            <!-- <slip1>1.0</slip1>
+            <slip2>1.0</slip2> -->
+          </ode>
+        </friction>
+      </surface>
+    </collision>
+  </link>
+  <!-- front wheel left connector -->
+  <link name="front_wheel_left_connector">
+    <inertial>
+      <origin
+        xyz="0 0 0"
+        rpy="0 0 0" />
+      <mass
+        value="0.1" />
+        <inertia
+          ixx="1E-3"
+          ixy="0"
+          ixz="0"
+          iyy="1E-3"
+          iyz="0"
+          izz="1E-3" />
+    </inertial>
+    <visual>
+      <origin
+        xyz="0 0 0"
+        rpy="0 0 0" />
+      <geometry>
+        <mesh
+          filename="package://fyp_sim/meshes/front_wheel_connector.stl" scale="0.01 0.01 0.01"/>
+      </geometry>
+      <material
+        name="front_wheel_left_connector_material">
+        <color
+          rgba="0.203125 0.238281 0.285156 1.0" />
+      </material>
+    </visual>
+    <!-- <collision name="front_wheel_left_connector_collision">
+      <origin
+        xyz="0 0 0"
+        rpy="0 0 0" />
+      <geometry>
+        <mesh
+          filename="package://fyp_sim/meshes/front_wheel_connector.stl" scale="0.01 0.01 0.01"/>
+      </geometry>
+    </collision> -->
+  </link>
+  <!-- front wheel left connector bar -->
+  <link name="front_wheel_left_bar">
+    <inertial>
+      <origin
+        xyz="-0.03 0 0"
+        rpy="0 0 0" />
+      <mass
+        value="0.1" />
+        <inertia
+          ixx="1E-3"
+          ixy="0"
+          ixz="0"
+          iyy="1E-3"
+          iyz="0"
+          izz="1E-3" />
+    </inertial>
+    <visual>
+      <origin
+        xyz="-0.03 0 0"
+        rpy="0 0 0" />
+      <geometry>
+        <box size="0.08 0.04 0.008"/>
+      </geometry>
+      <material
+        name="front_wheel_left_bar_material">
+        <color
+          rgba="0.203125 0.238281 0.285156 1.0" />
+      </material>
+    </visual>
+    <collision name="front_wheel_left_bar_collision">
+      <origin
+        xyz="-0.03 0 0"
+        rpy="0 0 0" />
+      <geometry>
+        <box size="0.08 0.04 0.008"/>
+      </geometry>
+    </collision>
+  </link>
+  <!-- front wheel right connector bar -->
+  <link name="front_wheel_right_bar">
+    <inertial>
+      <origin
+        xyz="-0.03 0 0"
+        rpy="0 0 0" />
+      <mass
+        value="0.1" />
+        <inertia
+          ixx="1E-3"
+          ixy="0"
+          ixz="0"
+          iyy="1E-3"
+          iyz="0"
+          izz="1E-3" />
+    </inertial>
+    <visual>
+      <origin
+        xyz="-0.03 0 0"
+        rpy="0 0 0" />
+      <geometry>
+        <box size="0.08 0.04 0.008"/>
+      </geometry>
+      <material
+        name="front_wheel_right_bar_material">
+        <color
+          rgba="0.203125 0.238281 0.285156 1.0" />
+      </material>
+    </visual>
+    <collision name="front_wheel_right_bar_collision">
+      <origin
+        xyz="-0.03 0 0"
+        rpy="0 0 0" />
+      <geometry>
+        <box size="0.08 0.04 0.008"/>
+      </geometry>
+    </collision>
+  </link>
+  <!-- front wheel right connector -->
+  <link name="front_wheel_right_connector">
+    <inertial>
+      <origin
+        xyz="0 0 0"
+        rpy="0 0 0" />
+      <mass
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