Commit message: Added odom node; tf data is not fixed

File: catkin_ws/src/fyp_sim/urdf/robot.xacro (robot description, xacro)
@@ -356,9 +356,9 @@
       link="back_wheel_right" />
     <axis
-      xyz="0 0 1" />
+      xyz="0 0 -1" />
   </joint>
   <joint name="front_LW_con_joint"
     type="revolute">
-    <limit effort="30" velocity="4.0" lower="-3.14159" upper="3.14159"/>
+    <limit effort="30" velocity="${pi}" lower="${-pi/3}" upper="${pi/3}"/>
     <origin
       xyz="-0.35409 -0.22 0.02013"
@@ -373,5 +373,5 @@
   <joint name="front_RW_con_joint"
     type="revolute">
-    <limit effort="30" velocity="4.0" lower="-3.14159" upper="3.14159"/>
+    <limit effort="30" velocity="${pi}" lower="${-pi/3}" upper="${pi/3}"/>
     <origin
       xyz="-0.35409 0.22 0.02013"

Commit message: Fixed tf data; added new transmission tags for front wheels

File: catkin_ws/src/fyp_sim/urdf/robot.xacro (robot description, xacro)
@@ -449,3 +449,24 @@
     </actuator>
   </transmission>
+  <!--For caster wheels; not for physical robot; only for simulation -->
+  <transmission name="front_RW_transmission">
+    <type>transmission_interface/SimpleTransmission</type>
+    <joint name="front_RW_joint">
+      <hardwareInterface>hardware_interface/EffortJointInterface</hardwareInterface>
+    </joint>
+    <actuator name="front_RW_motor">
+      <mechanicalReduction>1</mechanicalReduction>
+      <hardwareInterface>EffortJointInterface</hardwareInterface>
+    </actuator>
+  </transmission>
+  <transmission name="front_LW_transmission">
+    <type>transmission_interface/SimpleTransmission</type>
+    <joint name="front_LW_joint">
+      <hardwareInterface>hardware_interface/EffortJointInterface</hardwareInterface>
+    </joint>
+    <actuator name="front_LW_motor">
+      <mechanicalReduction>1</mechanicalReduction>
+      <hardwareInterface>EffortJointInterface</hardwareInterface>
+    </actuator>
+  </transmission>
 </robot>

Commit message: Added ekf_localization; added gps+wheel_odom+imu; tested ackerman

File: catkin_ws/src/fyp_sim/urdf/robot.xacro (robot description, xacro)
@@ -38,5 +38,5 @@
       <origin
         xyz="0 0 0"
-        rpy="0 0 0" />
+        rpy="0 0 ${-pi/2}" />
       <geometry>
         <mesh
@@ -328,5 +328,5 @@
     <origin
       xyz="0 0 0.22987"
-      rpy="0 0 0" />
+      rpy="0 0 ${-pi}" />
     <parent
       link="base_footprint" />
@@ -360,5 +360,5 @@
   <joint name="front_LW_con_joint"
     type="revolute">
-    <limit effort="30" velocity="${pi}" lower="${-pi/3}" upper="${pi/3}"/>
+    <limit effort="30" velocity="${pi/3}" lower="${-pi/2}" upper="${pi/2}"/>
     <origin
       xyz="-0.35409 -0.22 0.02013"
@@ -373,5 +373,5 @@
   <joint name="front_RW_con_joint"
     type="revolute">
-    <limit effort="30" velocity="${pi}" lower="${-pi/3}" upper="${pi/3}"/>
+    <limit effort="30" velocity="${pi/3}" lower="${-pi/2}" upper="${pi/2}"/>
     <origin
       xyz="-0.35409 0.22 0.02013"

Commit message: Changed front and back

File: catkin_ws/src/fyp_sim/urdf/robot.xacro (robot description, xacro)
@@ -46,5 +46,5 @@
   </link>
   <!-- back wheel left -->
-  <link name="back_wheel_left">
+  <link name="front_wheel_right">
     <inertial>
       <origin
@@ -96,5 +96,5 @@
   </link>
   <!-- back wheel right -->
-  <link name="back_wheel_right">
+  <link name="front_wheel_left">
     <inertial>
       <origin
@@ -146,5 +146,5 @@
   </link>
   <!-- front wheel left connector -->
-  <link name="front_wheel_left_connector">
+  <link name="back_wheel_right_connector">
     <inertial>
       <origin
@@ -186,5 +186,5 @@
   </link>
   <!-- front wheel left connector bar -->
-  <link name="front_wheel_left_bar">
+  <link name="back_wheel_right_bar">
     <inertial>
       <origin
@@ -224,5 +224,5 @@
   </link>
   <!-- front wheel right connector bar -->
-  <link name="front_wheel_right_bar">
+  <link name="back_wheel_left_bar">
     <inertial>
       <origin
@@ -262,5 +262,5 @@
   </link>
   <!-- front wheel right connector -->
-  <link name="front_wheel_right_connector">
+  <link name="back_wheel_left_connector">
     <inertial>
       <origin
@@ -302,5 +302,5 @@
   </link>
   <!-- front wheel right -->
-  <link name="front_wheel_right">
+  <link name="back_wheel_left">
     <inertial>
       <origin
@@ -352,5 +352,5 @@
   </link>
   <!-- front wheel left -->
-  <link name="front_wheel_left">
+  <link name="back_wheel_right">
     <inertial>
       <origin
@@ -401,5 +401,5 @@
     </collision>
   </link>
-  <link name="lidar">
+  <!-- <link name="lidar">
     <inertial>
       <origin
@@ -437,12 +437,9 @@
         </geometry>
     </collision>
-  </link>
+  </link> -->
   <joint name="base_joint" type="fixed">
     <origin
       xyz="0 0 0.22987"
-      rpy="0 0 ${pi}" />
-      <!-- <origin
-        xyz="0 0 0.22987"
-        rpy="0 0 0" /> -->
+      rpy="0 0 0" />
     <parent
       link="base_footprint" />
@@ -450,5 +447,5 @@
       link="chassis" />
   </joint>
-  <joint name="lidar_joint" type="fixed">
+  <!-- <joint name="lidar_joint" type="fixed">
     <origin
       xyz="-0.29 0 0.29"
@@ -458,119 +455,160 @@
     <child
       link="lidar" />
+  </joint> -->
+  <joint name="front_RW_joint"
+    type="continuous">
+    <origin
+      xyz="0.23591 -0.245 -0.06987"
+      rpy="${pi/2} 0 0" />
+    <parent
+      link="chassis" />
+    <child
+      link="front_wheel_right" />
+    <axis
+      xyz="0 0 -1" />
+      <dynamics friction="0.3"/>
+  </joint>
+  <joint name="front_LW_joint"
+    type="continuous">
+    <origin
+      xyz="0.23591 0.245 -0.06987"
+      rpy="${-pi/2} 0 0" />
+    <parent
+      link="chassis" />
+    <child
+      link="front_wheel_left" />
+    <axis
+      xyz="0 0 1" />
+      <dynamics friction="0.3"/>
+  </joint>
+  <joint name="back_wheel_right_bar_joint"
+    type="continuous">
+    <!-- <limit effort="30" velocity="${pi/3}" lower="${-pi/2}" upper="${pi/2}"/> -->
+    <origin
+      xyz="-0.35409 -0.22 -0.03"
+      rpy="0 0 0" />
+    <parent
+      link="chassis" />
+    <child
+      link="back_wheel_right_bar" />
+    <axis
+      xyz="0 0 1" />
+      <dynamics friction="0.2"/>
+  </joint>
+  <joint name="back_RW_con_joint"
+    type="fixed">
+    <!-- <limit effort="30" velocity="${pi/3}" lower="${-pi/2}" upper="${pi/2}"/> -->
+    <origin
+      xyz="-0.06 0 0.03513"
+      rpy="0 0 ${pi/2}" />
+    <parent
+      link="back_wheel_right_bar" />
+    <child
+      link="back_wheel_right_connector" />
+      <!-- front_wheel_left_bar -->
+    <axis
+      xyz="0 0 1" />
+  </joint>
+  <joint name="back_wheel_left_bar_joint"
+    type="continuous">
+    <!-- <limit effort="30" velocity="${pi/3}" lower="${-pi/2}" upper="${pi/2}"/> -->
+    <origin
+      xyz="-0.35409 0.22 -0.03"
+      rpy="0 0 0" />
+    <parent
+      link="chassis" />
+    <child
+      link="back_wheel_left_bar" />
+    <axis
+      xyz="0 0 1" />
+      <dynamics friction="0.2"/>
+  </joint>
+  <joint name="back_LW_con_joint"
+    type="fixed">
+    <!-- <limit effort="30" velocity="${pi/3}" lower="${-pi/2}" upper="${pi/2}"/> -->
+    <origin
+      xyz="-0.06 0 0.03513"
+      rpy="0 0 ${pi/2}" />
+    <parent
+      link="back_wheel_left_bar" />
+    <child
+      link="back_wheel_left_connector" />
+    <axis
+      xyz="0 0 1" />
   </joint>
   <joint name="back_LW_joint"
     type="continuous">
     <origin
-      xyz="0.23591 -0.245 -0.06987"
-      rpy="${pi/2} 0 0" />
-    <parent
-      link="chassis" />
+      xyz="0 0 -0.15"
+      rpy="0 ${pi/2} 0" />
+    <parent
+      link="back_wheel_left_connector" />
     <child
       link="back_wheel_left" />
     <axis
-      xyz="0 0 1" />
-      <dynamics friction="0.3"/>
-  </joint>
+      xyz="0 0 -1" />
+  </joint>
+<!-- "-0.35409 -0.22 -0.13487" -->
   <joint name="back_RW_joint"
     type="continuous">
     <origin
-      xyz="0.23591 0.245 -0.06987"
-      rpy="${-pi/2} 0 0" />
-    <parent
-      link="chassis" />
-    <child
-      link="back_wheel_right" />
-    <axis
-      xyz="0 0 -1" />
-      <dynamics friction="0.3"/>
-  </joint>
-  <joint name="front_wheel_left_bar_joint"
-    type="continuous">
-    <!-- <limit effort="30" velocity="${pi/3}" lower="${-pi/2}" upper="${pi/2}"/> -->
-    <origin
-      xyz="-0.35409 -0.22 -0.03"
-      rpy="0 0 ${pi}" />
-    <parent
-      link="chassis" />
-    <child
-      link="front_wheel_left_bar" />
-    <axis
-      xyz="0 0 1" />
-      <dynamics friction="0.2"/>
-  </joint>
-  <joint name="front_LW_con_joint"
-    type="fixed">
-    <!-- <limit effort="30" velocity="${pi/3}" lower="${-pi/2}" upper="${pi/2}"/> -->
-    <origin
-      xyz="-0.06 0 0.03513"
-      rpy="0 0 ${pi/2}" />
-    <parent
-      link="front_wheel_left_bar" />
-    <child
-      link="front_wheel_left_connector" />
-      <!-- front_wheel_left_bar -->
-    <axis
-      xyz="0 0 1" />
-  </joint>
-  <joint name="front_wheel_right_bar_joint"
-    type="continuous">
-    <!-- <limit effort="30" velocity="${pi/3}" lower="${-pi/2}" upper="${pi/2}"/> -->
-    <origin
-      xyz="-0.35409 0.22 -0.03"
-      rpy="0 0 ${pi}" />
-    <parent
-      link="chassis" />
-    <child
-      link="front_wheel_right_bar" />
-    <axis
-      xyz="0 0 1" />
-      <dynamics friction="0.2"/>
-  </joint>
-  <joint name="front_RW_con_joint"
-    type="fixed">
-    <!-- <limit effort="30" velocity="${pi/3}" lower="${-pi/2}" upper="${pi/2}"/> -->
-    <origin
-      xyz="-0.06 0 0.03513"
-      rpy="0 0 ${pi/2}" />
-    <parent
-      link="front_wheel_right_bar" />
-    <child
-      link="front_wheel_right_connector" />
-    <axis
-      xyz="0 0 1" />
-  </joint>
-  <joint name="front_RW_joint"
-    type="continuous">
-    <origin
-      xyz="0 0 -0.15"
-      rpy="0 ${pi/2} 0" />
-    <parent
-      link="front_wheel_right_connector" />
-    <child
-      link="front_wheel_right" />
-    <axis
-      xyz="0 0 -1" />
-  </joint>
-<!-- "-0.35409 -0.22 -0.13487" -->
-  <joint name="front_LW_joint"
-    type="continuous">
-    <origin
       xyz="0 0 -0.15"
       rpy="0 ${-pi/2} 0" />
     <parent
-      link="front_wheel_left_connector"/>
-    <child
-      link="front_wheel_left" />
+      link="back_wheel_right_connector"/>
+    <child
+      link="back_wheel_right" />
     <axis
       xyz="0 0 1" />
   </joint>
+  <transmission name="front_RW_transmission">
+    <type>transmission_interface/SimpleTransmission</type>
+    <joint name="front_RW_joint">
+      <hardwareInterface>hardware_interface/VelocityJointInterface</hardwareInterface>
+    </joint>
+    <actuator name="front_RW_motor">
+      <mechanicalReduction>1</mechanicalReduction>
+      <hardwareInterface>VelocityJointInterface</hardwareInterface>
+    </actuator>
+  </transmission>
+  <transmission name="front_LW_transmission">
+    <type>transmission_interface/SimpleTransmission</type>
+    <joint name="front_LW_joint">
+      <hardwareInterface>hardware_interface/VelocityJointInterface</hardwareInterface>
+    </joint>
+    <actuator name="front_LW_motor">
+      <mechanicalReduction>1</mechanicalReduction>
+      <hardwareInterface>VelocityJointInterface</hardwareInterface>
+    </actuator>
+  </transmission>
+  <transmission name="back_wheel_left_bar_transmission">
+    <type>transmission_interface/SimpleTransmission</type>
+    <joint name="back_wheel_left_bar_joint">
+      <hardwareInterface>hardware_interface/EffortJointInterface</hardwareInterface>
+    </joint>
+    <actuator name="back_wheel_left_bar_motor">
+      <mechanicalReduction>1</mechanicalReduction>
+      <hardwareInterface>EffortJointInterface</hardwareInterface>
+    </actuator>
+  </transmission>
+  <transmission name="back_wheel_right_bar_transmission">
+    <type>transmission_interface/SimpleTransmission</type>
+    <joint name="back_wheel_right_bar_joint">
+      <hardwareInterface>hardware_interface/EffortJointInterface</hardwareInterface>
+    </joint>
+    <actuator name="back_wheel_right_bar_motor">
+      <mechanicalReduction>1</mechanicalReduction>
+      <hardwareInterface>EffortJointInterface</hardwareInterface>
+    </actuator>
+  </transmission>
+  <!--For caster wheels; not for physical robot; only for simulation -->
   <transmission name="back_LW_transmission">
     <type>transmission_interface/SimpleTransmission</type>
     <joint name="back_LW_joint">
-      <hardwareInterface>hardware_interface/VelocityJointInterface</hardwareInterface>
+      <hardwareInterface>hardware_interface/EffortJointInterface</hardwareInterface>
     </joint>
     <actuator name="back_LW_motor">
       <mechanicalReduction>1</mechanicalReduction>
-      <hardwareInterface>VelocityJointInterface</hardwareInterface>
+      <hardwareInterface>EffortJointInterface</hardwareInterface>
     </actuator>
   </transmission>
@@ -578,48 +616,7 @@
     <type>transmission_interface/SimpleTransmission</type>
     <joint name="back_RW_joint">
-      <hardwareInterface>hardware_interface/VelocityJointInterface</hardwareInterface>
+      <hardwareInterface>hardware_interface/EffortJointInterface</hardwareInterface>
     </joint>
     <actuator name="back_RW_motor">
-      <mechanicalReduction>1</mechanicalReduction>
-      <hardwareInterface>VelocityJointInterface</hardwareInterface>
-    </actuator>
-  </transmission>
-  <transmission name="front_wheel_right_bar_transmission">
-    <type>transmission_interface/SimpleTransmission</type>
-    <joint name="front_wheel_right_bar_joint">
-      <hardwareInterface>hardware_interface/EffortJointInterface</hardwareInterface>
-    </joint>
-    <actuator name="front_wheel_right_bar_motor">
-      <mechanicalReduction>1</mechanicalReduction>
-      <hardwareInterface>EffortJointInterface</hardwareInterface>
-    </actuator>
-  </transmission>
-  <transmission name="front_wheel_left_bar_transmission">
-    <type>transmission_interface/SimpleTransmission</type>
-    <joint name="front_wheel_left_bar_joint">
-      <hardwareInterface>hardware_interface/EffortJointInterface</hardwareInterface>
-    </joint>
-    <actuator name="front_wheel_left_bar_motor">
-      <mechanicalReduction>1</mechanicalReduction>
-      <hardwareInterface>EffortJointInterface</hardwareInterface>
-    </actuator>
-  </transmission>
-  <!--For caster wheels; not for physical robot; only for simulation -->
-  <transmission name="front_RW_transmission">
-    <type>transmission_interface/SimpleTransmission</type>
-    <joint name="front_RW_joint">
-      <hardwareInterface>hardware_interface/EffortJointInterface</hardwareInterface>
-    </joint>
-    <actuator name="front_RW_motor">
-      <mechanicalReduction>1</mechanicalReduction>
-      <hardwareInterface>EffortJointInterface</hardwareInterface>
-    </actuator>
-  </transmission>
-  <transmission name="front_LW_transmission">
-    <type>transmission_interface/SimpleTransmission</type>
-    <joint name="front_LW_joint">
-      <hardwareInterface>hardware_interface/EffortJointInterface</hardwareInterface>
-    </joint>
-    <actuator name="front_LW_motor">
       <mechanicalReduction>1</mechanicalReduction>
       <hardwareInterface>EffortJointInterface</hardwareInterface>
